File: board/board.kicad_pcb (KiCad board)
At the start: 2 copper layers, 21 x 13 mm, 1 part

Commit message: initial
Parts:
- added D1: ABS2, Diode_SMD:Diode_Bridge_Diotec_ABS, F.Cu at (150.2, 94.1)
- added D2: ABS2, Diode_SMD:Diode_Bridge_Diotec_ABS, F.Cu at (150.2, 99.6)
- added J1: 004_BASE-T_CT, on_edge:on_edge_2x05_device, F.Cu at (140.0, 96.5)
- added J2: 013_PoE_rectified, on_edge:on_edge_2x05_host, F.Cu at (161.0, 96.5)
- LOGO1: moved to B.Cu
- turned LOGO1 to 180 degrees
Routing:
- net /rectifier/-: track 0.00 -> 18.5 mm, vias 0 -> 2
- net /rectifier/+: track 0.00 -> 17.9 mm
- net GND: track 0.00 -> 17.3 mm
- net /5V: track 0.00 -> 16.2 mm
- net /3.3V: track 0.00 -> 16.2 mm
- net /rectifier1/~1: track 0.00 -> 11.9 mm
- net /rectifier/~2: track 0.00 -> 7.22 mm, vias 0 -> 1
- net /rectifier/~1: track 0.00 -> 6.85 mm, vias 0 -> 1
- net /rectifier1/~2: track 0.00 -> 5.27 mm
Other:
- outline, holes or cut-outs redrawn
- board text added: "osf.004"
- board text added: "osf.013"
- board text added: "osf.b157.v1.0"
